File: electronics/5vbuck/5vbuck.kicad_pcb (KiCad board)
At the start: 2 copper layers, 10 parts, among them J1 in, J2 USB_A, J3 out, U1 LM2596S-5

Commit message: irduino small board design
Routing:
- net Net-(C1-Pad2): track 101.7 -> 128.8 mm
- net Net-(C1-Pad1): track 48.1 -> 52.8 mm
- removed copper zone on B.Cu, net Net-(C1-Pad2)
Other:
- net class Default: clearance 0.5 -> 0.7; trace_width 1 -> 1.5
- rule trace_clearance: 0.5 -> 0.7
Changed lines of the file:
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@@
     (thickness 1.6)
     (drawings 0)
-    (tracks 45)
+    (tracks 51)
     (zones 0)
     (modules 10)
@@
   )
   (setup
-    (last_trace_width 1)
-    (trace_clearance 0.5)
+    (last_trace_width 1.5)
+    (trace_clearance 0.7)
     (zone_clearance 0.508)
     (zone_45_only no)
@@
   (net 5 "Net-(J2-Pad5)")
   (net_class Default "This is the default net class."
-    (clearance 0.5)
-    (trace_width 1)
+    (clearance 0.7)
+    (trace_width 1.5)
     (via_dia 0.8)
     (via_drill 0.4)
@@
   (segment (start 97.79 90.852) (end 108.966 90.852) (width 1.5) (layer B.Cu) (net 1))
   (segment (start 87.63 90.852) (end 97.79 90.852) (width 1.5) (layer B.Cu) (net 1))
-  (segment (start 86.44 89.662) (end 87.63 90.852) (width 1.5) (layer B.Cu) (net 1))
-  (segment (start 76.962 89.662) (end 86.44 89.662) (width 1.5) (layer B.Cu) (net 1))
   (segment (start 87.769 76.157) (end 87.769 75.457) (width 1.5) (layer B.Cu) (net 1))
   (segment (start 93.969 82.357) (end 87.769 76.157) (width 1.5) (layer B.Cu) (net 1))
@@
   (segment (start 120.538 69.2) (end 125.984 69.2) (width 1.5) (layer B.Cu) (net 1))
   (segment (start 119.634 70.104) (end 120.538 69.2) (width 1.5) (layer B.Cu) (net 1))
+  (segment (start 131.202 90.286) (end 130.302 91.186) (width 1.5) (layer B.Cu) (net 1))
+  (segment (start 133.55201 87.93599) (end 131.202 90.286) (width 1.5) (layer B.Cu) (net 1))
+  (segment (start 127.11537 69.2) (end 133.55201 75.63664) (width 1.5) (layer B.Cu) (net 1))
+  (segment (start 133.55201 75.63664) (end 133.55201 87.93599) (width 1.5) (layer B.Cu) (net 1))
+  (segment (start 125.984 69.2) (end 127.11537 69.2) (width 1.5) (layer B.Cu) (net 1))
+  (segment (start 78.152 90.852) (end 76.962 89.662) (width 1.5) (layer B.Cu) (net 1))
+  (segment (start 87.63 90.852) (end 78.152 90.852) (width 1.5) (layer B.Cu) (net 1))
   (segment (start 78.232 85.852) (end 76.962 84.582) (width 1.5) (layer B.Cu) (net 2))
   (segment (start 87.63 85.852) (end 78.232 85.852) (width 1.5) (layer B.Cu) (net 2))
-  (segment (start 96.919 72.057) (end 97.028 71.374) (width 1) (layer B.Cu) (net 2))
-  (segment (start 76.962 84.582) (end 76.962 72.898) (width 1.5) (layer B.Cu) (net 2))
-  (segment (start 97.028 69.088) (end 97.028 71.374) (width 1.5) (layer B.Cu) (net 2))
-  (segment (start 96.266 68.326) (end 97.028 69.088) (width 1.5) (layer B.Cu) (net 2))
-  (segment (start 76.962 72.898) (end 81.534 68.326) (width 1.5) (layer B.Cu) (net 2))
-  (segment (start 81.534 68.326) (end 96.266 68.326) (width 1.5) (layer B.Cu) (net 2))
+  (segment (start 85.33 85.852) (end 79.502 80.024) (width 1.5) (layer B.Cu) (net 2))
+  (segment (start 87.63 85.852) (end 85.33 85.852) (width 1.5) (layer B.Cu) (net 2))
+  (segment (start 79.502 80.024) (end 79.502 70.104) (width 1.5) (layer B.Cu) (net 2))
+  (segment (start 79.502 70.104) (end 81.534 68.072) (width 1.5) (layer B.Cu) (net 2))
+  (segment (start 81.534 68.072) (end 95.504 68.072) (width 1.5) (layer B.Cu) (net 2))
+  (segment (start 96.919 69.487) (end 96.919 71.756999) (width 1.5) (layer B.Cu) (net 2))
+  (segment (start 95.504 68.072) (end 96.919 69.487) (width 1.5) (layer B.Cu) (net 2))
   (segment (start 130.128 85.932) (end 130.302 86.106) (width 1.5) (layer B.Cu) (net 3))
   (segment (start 117.348 85.932) (end 130.128 85.932) (width 1.5) (layer B.Cu) (net 3))
@@
   (segment (start 96.919 73.757) (end 102.941 73.757) (width 1) (layer B.Cu) (net 4))
   (segment (start 104.394 78.74) (end 104.394 70.104) (width 1.5) (layer B.Cu) (net 4))
-  (zone (net 1) (net_name "Net-(C1-Pad2)") (layer B.Cu) (hatch edge 0.508)
-    (connect_pads (clearance 0.508))
-    (min_thickness 0.254)
-    (fill yes (arc_segments 32) (thermal_gap 0.508) (thermal_bridge_width 0.508))
-    (polygon
-      (pts
-        (xy 140.462 94.742) (xy 72.644 94.742) (xy 72.898 62.738) (xy 140.462 62.738)
-      )
-    )
-  )
 )
