File: electronics/simple-charger/simple-charger.sch (KiCad schematic (older format))
At the start: 43 parts, among them J1 SolarPanel, J2 LoadConnector, J3 BatteryTerminal, J4 IR Switch, J5 SPI, J6 USB_A, Q1 IRLIZ44N, Q2 IRLIZ44N, Q3 IRLIZ44N, Q4 IRLIZ44N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

Commit message: PCB design
Parts:
- removed Q5, Q6: BSS138, Package_TO_SOT_SMD:SOT-23, symbol Transistor_FET:BSS138
- added J7: refJUMPER, Connector_PinHeader_2.54mm:PinHeader_1x02_P2.54mm_Vertical, symbol Connector:Conn_01x02_Male
- added Q5, Q6: BC307, Package_TO_SOT_THT:TO-92L_Wide, symbol Transistor_BJT:BC307
- added R17, R18: 10k, Resistor_THT:R_Axial_DIN0204_L3.6mm_D1.6mm_P7.62mm_Horizontal, symbol Device:R
- added R19: 1.7k, Resistor_THT:R_Axial_DIN0204_L3.6mm_D1.6mm_P7.62mm_Horizontal, symbol Device:R
- added U5: TL431DBZ, Package_TO_SOT_SMD:SOT-23, symbol Reference_Voltage:TL431DBZ
Connections:
- net +5V: now also J7.2 (Pin_2)
- net BatteryPowerSensor: now also A1.21 (A2); no longer A1.19 (A0)
- net ChargeEnable: now also ULN2003A1.16 (O1), Q6.2 (B), R18.1; no longer A1.8 (D5)
- net GND: now also Q4.3 (S), U5.3 (A)
- net LoadEnable: now also ULN2003A1.15 (O2), Q5.2 (B), R17.1; no longer A1.9 (D6)
- net PWR: now also Q5.3 (E), Q6.3 (E), R17.2, R18.2; no longer Q4.3 (S)
- net SolarPowerSensor: now also A1.19 (A0); no longer A1.21 (A2)
- net at A1.18 (AREF): now also R19.2, U5.1 (K), U5.2 (REF)
- net at A1.5 (D2): now also ULN2003A1.4 (I4); no longer ULN2003A1.1 (I1)
- net at A1.6 (D3): now also ULN2003A1.3 (I3); no longer ULN2003A1.2 (I2)
- net at A1.7 (D4): now also ULN2003A1.2 (I2); no longer J4.3 (Pin_3)
- net at ULN2003A1.13 (O4): now also J4.2 (Pin_2)
- net at ULN2003A1.14 (O3): now also J4.3 (Pin_3)
- net at J4.1 (Pin_1): now also A1.9 (D6); no longer ULN2003A1.16 (O1)
- net at R12.1: now also Q6.1 (C)
- net at R16.1: now also Q5.1 (C)
- new net: A1.8 (D5), ULN2003A1.1 (I1)
- new net: J7.1 (Pin_1), R19.1
- no-connect marks 32 -> 27
